File: hardware/IOBoard2021/IOBoard2021.kicad_pcb (KiCad board)
At the start: 2 copper layers, 86 x 66 mm, 66 parts, among them J1 SERVO, J10 PUMP, J11 EV, J12 PRESSURE, J13 PRESSURE, J14 PRESSURE, J15 DISPLAY, J16 PUMP, J17 EV, J18 UART, J19 I2C, J2 SERVO, J20 STEPPER, J21 Rmeas, J22 HMI, J23 STEPPER, J3 FDC, J4 FDC, J5 PUMP, J6 EV, J7 22-03-5035, J8 22-03-5035, J9 Screw_Terminal_01x02, U1 IRLML6344, U10 TCA9554DBQ, U11 TCA9554DBQ, U2 IRLML6344, U3 TSR_1-2450, U4 LM3940_IMP3.3, U5 IRLML6344, U6 IRLML6344, U7 IRLML6344, U8 IRLML6344, U9 NUCLEO32-L432KC

Commit message: Finish board.
Parts:
- added G***: RustyDucks, myFootprints:RustyDuck, B.Cu at (124.5, 88.1)
- added REF**: USB_LOGO, myFootprints:USB_LOGO, F.Cu at (120.7, 70.9)
Routing:
- net +5V: track 134.7 -> 131.2 mm
- net +3V3: track 175.8 -> 176.8 mm
- net R_MEAS: track 62.7 -> 62.1 mm
- added copper zone on F.Cu, net GND
Other:
- board text added: "12V"
- board text added: "1A"
- board text added: "1B"
- board text added: "2A"
- board text added: "2B"
- board text added: "AX12"
- board text added: "B"
- board text added: "Bt."
- board text added: "Col."
- board text added: "DISPLAY"
- board text added: "EV1"
- board text added: "EV2"
- board text added: "EV3"
- board text added: "FDC1"
- board text added: "FDC2"
- board text added: "Fab@TheRustyDucks 2022"
- board text added: "G"
- board text added: "GND"
- board text added: "HMI"
- board text added: "I2C"
- board text added: "IO board 2022"
- board text added: "NucleoL432"
- board text added: "POWER"
- board text added: "PRESSURE1"
- board text added: "PRESSURE2"
- board text added: "PRESSURE3"
- board text added: "PUMP1"
- board text added: "PUMP2"
- board text added: "PUMP3"
- board text added: "R"
- board text added: "SERVO1"
- board text added: "SERVO2"
- board text added: "STEP.1"
- board text added: "STEP.2"
- board text added: "Tir."
- board text added: "UART"
- board text added: "Ω"
