File: hardware/IOBoard2021/IOBoard2021.kicad_sch (KiCad schematic)
At the start: 5 parts

Commit message: Finish schematic and copper layout.
Parts:
- removed U?: PCA9555D, Package_SO:SOIC-24W_7.5x15.4mm_P1.27mm, symbol Interface_Expansion:PCA9555D
- added A1, A2: Pololu_Breakout_A4988, Module:Pololu_Breakout-16_15.2x20.3mm, symbol Driver_Motor:Pololu_Breakout_A4988
- added C1: 470n, Capacitor_SMD:C_0603_1608Metric_Pad1.08x0.95mm_HandSolder, symbol Device:C_Small
- added C10, C6: 100u, Capacitor_Tantalum_SMD:CP_EIA-7343-31_Kemet-D_Pad2.25x2.55mm_HandSolder, symbol Device:C_Polarized
- added C2, C3, C4: 10u, Capacitor_SMD:C_0603_1608Metric_Pad1.08x0.95mm_HandSolder, symbol Device:C_Small
- added C5, C7, C8, C9: 100n, Capacitor_SMD:C_0603_1608Metric_Pad1.08x0.95mm_HandSolder, symbol Device:C_Small
- added D1, D2, D3, D4, D5, D6: PMEG2020EH, Diode_SMD:D_SOD-123F, symbol Diode:PMEG2020EH
- added J1, J2: SERVO, Connector_PinHeader_2.54mm:PinHeader_1x03_P2.54mm_Vertical, symbol Connector:Conn_01x03_Male
- added J10, J16, J5: PUMP, Connector_PinHeader_2.54mm:PinHeader_1x02_P2.54mm_Vertical_SMD_Pin1Left, symbol Connector:Conn_01x02_Male
- added J11, J17, J6: EV, Connector_PinHeader_2.54mm:PinHeader_1x02_P2.54mm_Vertical_SMD_Pin1Left, symbol Connector:Conn_01x02_Male
- added J12, J13, J14: PRESSURE, Connector_Molex:Molex_PicoBlade_53398-0471_1x04-1MP_P1.25mm_Vertical, symbol Connector:Conn_01x04_Male
- added J15: DISPLAY, Connector_Molex:Molex_PicoBlade_53398-0471_1x04-1MP_P1.25mm_Vertical, symbol Connector:Conn_01x04_Male
- added J18: UART, Connector_Molex:Molex_PicoBlade_53398-0471_1x04-1MP_P1.25mm_Vertical, symbol Connector:Conn_01x04_Male
- added J19: I2C, Connector_Molex:Molex_PicoBlade_53398-0471_1x04-1MP_P1.25mm_Vertical, symbol Connector:Conn_01x04_Male
- added J20, J23: STEPPER, Connector_PinHeader_2.54mm:PinHeader_1x04_P2.54mm_Vertical, symbol Connector:Conn_01x04_Male
- added J21: Rmeas, Connector_PinHeader_2.54mm:PinHeader_1x02_P2.54mm_Vertical, symbol Connector:Conn_01x02_Male
- added J3, J4: FDC, Connector_PinHeader_2.54mm:PinHeader_1x02_P2.54mm_Vertical, symbol Connector:Conn_01x02_Male
- added J7, J8: 22-03-5035, myFootprints:SHDR3W70P0X250_1X3_990X490X590P, symbol mySymbols:22-03-5035
- added J9: Screw_Terminal_01x02, TerminalBlock:TerminalBlock_bornier-2_P5.08mm, symbol Connector:Screw_Terminal_01x02
- added R1, R2, R3, R4, R5, R6: 10k, Resistor_SMD:R_0603_1608Metric_Pad0.98x0.95mm_HandSolder, symbol Device:R
- added R10: 4.7k, Resistor_SMD:R_0603_1608Metric_Pad0.98x0.95mm_HandSolder, symbol Device:R
- added R7: 1k, Resistor_SMD:R_0603_1608Metric_Pad0.98x0.95mm_HandSolder, symbol Device:R
- added U1, U2, U5, U6, U7, U8: IRLML6344, myFootprints:SOT-23, symbol mySymbols:IRLML6344
- added U10, U11: TCA9554DBQ, Package_SO:SSOP-16_3.9x4.9mm_P0.635mm, symbol Interface_Expansion:TCA9554DBQ
- added U3: TSR_1-2450, Converter_DCDC:Converter_DCDC_TRACO_TSR-1_THT, symbol Regulator_Switching:TSR_1-2450
- added U4: LM3940_IMP3.3, Package_TO_SOT_SMD:SOT-223-3_TabPin2, symbol mySymbols:LM3940_IMP3.3
- J22: renamed from J?; footprint (none) -> Connector_IDC:IDC-Header_2x04_P2.54mm_Vertical
- R8, R9: renamed from R?; footprint (none) -> Resistor_SMD:R_0603_1608Metric_Pad0.98x0.95mm_HandSolder
- gave numbers to parts that had none: 1
Connections:
- net SERVO3 is gone; now on net PDIR2: U9.9 (PB01)
- net SERVO4 is gone; now on net PDIR1: U9.6 (PB00)
- net +3V3: now also U9.17 (+3V3), A1.10 (MS1), A1.11 (MS2), A1.2 (VDD), A2.10 (MS1), A2.11 (MS2), A2.2 (VDD), C2.1, C3.1, C4.1, C5.2, C7.2, C8.2, C9.2, R10.1, R7.1, U10.16 (VDD), U11.1 (A0), U11.16 (VDD), U4.3 (VOUT)
- net BUTTON: now also J22.3 (Pin_3), U10.9 (P4); no longer J22.4 (Pin_4)
- net COLOR: now also J22.8 (Pin_8), U10.4 (P0); no longer J22.3 (Pin_3)
- net DISPLAY_CLK: now also J15.4 (Pin_4)
- net DISPLAY_DIO: now also J15.3 (Pin_3)
- net Dynamixel: now also J7.3, J8.3
- net EV1: now also R2.1, U11.7 (P3), U2.1 (G)
- net EV2: now also R4.1, U11.10 (P5), U6.1 (G)
- net EV3: now also R6.1, U11.9 (P4), U8.1 (G)
- net FDC1: now also J3.2 (Pin_2), U10.12 (P7)
- net FDC2: now also J4.2 (Pin_2), U10.11 (P6)
- net GND: now also U9.29 (GND), U9.4 (GND), A1.1 (GND), A1.12 (MS3), A1.7 (GND), A2.1 (GND), A2.12 (MS3), A2.7 (GND), C1.2, C10.2, C2.2, C3.2, C4.2, C5.1, C6.2, C7.1, C8.1, C9.1, J1.1 (Pin_1), J12.2 (Pin_2), J13.2 (Pin_2), J14.2 (Pin_2), J15.2 (Pin_2), J18.2 (Pin_2), J19.2 (Pin_2), J2.1 (Pin_1), J21.1 (Pin_1), J3.1 (Pin_1), J4.1 (Pin_1), J7.1, J8.1, J9.1 (Pin_1), R1.2, R2.2, R3.2, R4.2, R5.2, R6.2, U1.2 (S), U10.1 (A0), U10.2 (A1), U10.3 (A2), U10.8 (GND), U11.2 (A1), U11.3 (A2), U11.8 (GND), U2.2 (S), U3.2 (GND), U4.2 (GND), U5.2 (S), U6.2 (S), U7.2 (S), U8.2 (S)
- net I2C1_SCL: now also J19.4 (Pin_4), U10.14 (SCL), U11.14 (SCL)
- net I2C1_SDA: now also J19.3 (Pin_3), U10.15 (SDA), U11.15 (SDA)
- net LEDB: now also J22.4 (Pin_4), U10.6 (P2); no longer J22.7 (Pin_7)
- net LEDG: now also U10.5 (P1)
- net LEDR: now also U10.10 (P5)
- net PDIR1: now also A1.16 (DIR)
- net PDIR2: now also A2.16 (DIR)
- net PEN1: now also A1.9 (~{ENABLE}), U11.11 (P6)
- net PEN2: now also A2.9 (~{ENABLE}), U11.12 (P7)
- net PRESSURE1: now also J12.4 (Pin_4)
- net PRESSURE2: now also J13.4 (Pin_4)
- net PRESSURE3: now also J14.4 (Pin_4)
- net PSTEP1: now also U9.20 (PA01), A1.15 (STEP); no longer U9.19 (PA00)
- net PSTEP2: now also U9.19 (PA00), A2.15 (STEP); no longer U9.20 (PA01)
- net PUMP1: now also R1.1, U1.1 (G), U11.4 (P0)
- net PUMP2: now also R3.1, U11.5 (P1), U5.1 (G)
- net PUMP3: now also R5.1, U11.6 (P2), U7.1 (G)
- net SERVO1: now also J1.3 (Pin_3)
- net SERVO2: now also J2.3 (Pin_3)
- net TIRETTE: now also U10.7 (P3)
- net UART2_RX: now also J18.4 (Pin_4)
- net UART2_TX: now also J18.3 (Pin_3)
- net R_MEAS: now reaches U9.22 (PA04)
- net R_MEAS: now also J21.2 (Pin_2), R7.2
- net PCA_INT renamed PRESSURE_CLK
- net PRESSURE_CLK: now also J12.3 (Pin_3), J13.3 (Pin_3), J14.3 (Pin_3); no longer U9.5 (PA12)
- new net: D6.2 (A), J17.2 (Pin_2), U8.3 (D)
- new net: A1.3 (1B), J20.1 (Pin_1)
- new net: A1.4 (1A), J20.2 (Pin_2)
- new net: A1.5 (2A), J20.3 (Pin_3)
- new net: A1.6 (2B), J20.4 (Pin_4)
- new net: D2.2 (A), J6.2 (Pin_2), U2.3 (D)
- new net: D1.2 (A), J5.2 (Pin_2), U1.3 (D)
- new net: D4.2 (A), J11.2 (Pin_2), U6.3 (D)
- new net: D3.2 (A), J10.2 (Pin_2), U5.3 (D)
- new net: A2.3 (1B), J23.1 (Pin_1)
- new net: A2.4 (1A), J23.2 (Pin_2)
- new net: A2.5 (2A), J23.3 (Pin_3)
- new net: A2.6 (2B), J23.4 (Pin_4)
- new net: D5.2 (A), J16.2 (Pin_2), U7.3 (D)
- new net +12V: A1.8 (VMOT), A2.8 (VMOT), C10.1, C6.1, D1.1 (K), D2.1 (K), D3.1 (K), D4.1 (K), D5.1 (K), D6.1 (K), J10.1 (Pin_1), J11.1 (Pin_1), J16.1 (Pin_1), J17.1 (Pin_1), J5.1 (Pin_1), J6.1 (Pin_1), J7.2, J8.2, J9.2 (Pin_2), U3.1 (Vin)
- new net +5V: C1.1, J1.2 (Pin_2), J12.1 (Pin_1), J13.1 (Pin_1), J14.1 (Pin_1), J15.1 (Pin_1), J18.1 (Pin_1), J19.1 (Pin_1), J2.2 (Pin_2), U3.3 (Vout), U4.1 (VIN)
- new net TCA_INT: R10.2, U10.13 (~{INT}), U9.5 (PA12)
- no-connect marks 6 -> 14
Other:
- moved on the sheet: J22, U9

Commit message: Finish board.
Other:
- company: (none) -> The Rusty Ducks
- title: (none) -> IO board 2022
Changed lines of the file:
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@@
 (kicad_sch (version 20211123) (generator eeschema)
   (paper "A3")
+  (title_block
+    (title "IO board 2022")
+    (date "2022-02-01")
+    (rev "R1")
+    (company "The Rusty Ducks")
+    (comment 1 "Fabien")
+  )
   (junction (at 248.92 140.97) (diameter 0) (color 0 0 0 0)
   )
